File: hardware/GERI_Gadget.brd (EAGLE design)
At the start: 33 x 42 mm, 62 parts, among them IC1 OP-SINGLEOT, Q1 5.8A/30V/35mΩ, Q2 5.8A/30V/35mΩ, U3 UG-2864HSWEG01, U4 ATSAMD21G-A, Y1 32.768kHz

Commit message: updates...almost done
Parts:
- removed ACCEL: LIS3DH, SparkFun-Sensors:LGA-16-3X3
- removed C26: 10uF, CalvEngIO-Passives:C0603
- removed C28, C29: 2.2uF, CalvEngIO-Passives:C0603
- removed CHRG: MCP73831, CalvEngIO-Power:SOT23-5
- removed D8, D9: (no value), CalvEngIO-DiscreteSemi:USC
- removed IC1: OP-SINGLEOT, CalvEngIO-AnalogIC:SOT23-5
- removed JP6: CORTEX_DEBUGPTH, samd21-temp:2X5-PTH-1.27MM
- removed LDO: MIC5504, CalvEngIO-Power:SOT23-5
- removed LIS3DH.ACCEL: (no value), CalvEngIO-Connectors:1X04
- removed R22: 10K, CalvEngIO-Passives:R0402-BIGGER
- removed R33: 390K, CalvEngIO-Passives:R0402-BIGGER
- removed U$1: BUZZER_CMT-6635C-030, CalvEngIO-Electromechanical:BUZZER_CMT-6635C-030
- removed U$15: USB.MICRO-BIGGERPADS, CalvEngIO-Connectors:USB-MICRO-01.BIGGERPADS
- added BUZZ1: BUZZER.GENERIC, CalvEngIO-Electromechanical:PIEZO-1
- added C13: 10uF, CalvEngIO-Passives:C0603
- added C20: 100n, CalvEngIO-Passives:C0402
- added C5: 0.1uF, CalvEngIO-Passives:C0402
- added D1, D3: (no value), CalvEngIO-DiscreteSemi:USC
- added J2: CORTEX_DEBUG_PTH, CalvEngIO-Connectors:2X5-PTH-1.27MM
- added J3: (no value), CalvEngIO-Connectors:1X04
- added LDO1: MIC5504, CalvEngIO-Power:SOT23-5
- added OP1: OP-SINGLEOT, CalvEngIO-AnalogIC:SOT23-5
- added R14: 10k, SparkFun-Resistors:0402
- added R17: PHOTOCELLPTH, CalvEngIO-Sensors:PHOTOCELL
- added REV1: REVISION.A, CalvEngIO-Logos:REV.A
- added U1: ATSAMD21G-A, CalvEngIO-Microcontrollers:TQFP-48
- added U2: MCP73831, CalvEngIO-Power:SOT23-5
- added USB1: USB.MICRO-BIGGERPADS, CalvEngIO-Connectors:USB-MICRO-01.BIGGERPADS
- C1: value 100n -> 0.1uF
- C12: value 0.1uF -> 100nF
- C14: value 10u -> 10uF
- C15, C16: value 2.2u -> 2.2uF
- C17: value 10u -> 2.2uF
- C18: value 0.1uF -> 2.2uF; device SparkFun-Capacitors:0402 -> CalvEngIO-Passives:C0603
- C2: value 100n -> 15pF
- C21: value 10uF -> 100n; device SparkFun-Capacitors:0603 -> CalvEngIO-Passives:C0402
- C22: value 2.2uF -> 0.1uF; device CalvEngIO-Passives:C0603 -> SparkFun-Capacitors:0402
- C23: value 2.2uF -> 10uF; device CalvEngIO-Passives:C0603 -> SparkFun-Capacitors:0603
- C3: value 10uF -> 15pF; device CalvEngIO-Passives:C0603 -> CalvEngIO-Passives:C0402
- C4: value 100nF -> 0.1uF
- C6: value 0.1uF -> 10u; device CalvEngIO-Passives:C0402 -> CalvEngIO-Passives:C0603
- C7: value 15pF -> 2.2u; device CalvEngIO-Passives:C0402 -> CalvEngIO-Passives:C0603
- C8: value 0.1uF -> 2.2u; device CalvEngIO-Passives:C0402 -> CalvEngIO-Passives:C0603
- C9: value 15pF -> 10u; device CalvEngIO-Passives:C0402 -> CalvEngIO-Passives:C0603
- R1: value 390k -> 10K
- R11: value 10K -> 390k
- R13: value 10k -> 1k
- R15: value 1k -> 10k; device CalvEngIO-Passives:R0402-BIGGER -> SparkFun-Resistors:0402
- R16: value 390k -> 10k
- R4: value 10k -> 10K
- R5: value 10k -> 390k; device SparkFun-Resistors:0402 -> CalvEngIO-Passives:R0402-BIGGER
- R6: value 10k -> 390K; device SparkFun-Resistors:0402 -> CalvEngIO-Passives:R0402-BIGGER
- R9: value PHOTOCELLPTH -> 10k; device CalvEngIO-Sensors:PHOTOCELL -> CalvEngIO-Passives:R0402-BIGGER
- U4: value ATSAMD21G-A -> LIS3DH; device samd21-temp:TQFP-48 -> SparkFun-Sensors:LGA-16-3X3
- moved C4 51.4 mm to (5.16, 16.7), flipped to the bottom, turned to 270 degrees
- moved C14 50.1 mm to (21.7, 9.72), turned to 180 degrees
- moved C17 48.1 mm to (7.76, 24.1), flipped to the top, turned to 90 degrees
- moved C15 47.3 mm to (9.66, 24.0), flipped to the top, turned to 90 degrees
- moved C11 44.7 mm to (6.87, 12.2)
- moved R16 41.6 mm to (23.3, 36.7), flipped to the bottom, turned to 90 degrees
- moved C12 41.5 mm to (22.9, 6.59), turned to 90 degrees
- moved C16 41.2 mm to (23.4, 24.2), flipped to the top, turned to 270 degrees
- moved Q1 38.5 mm to (19.9, 12.3), flipped to the bottom
- moved C3 37.5 mm to (8.98, 24.2), flipped to the bottom
- moved R13 36.7 mm to (6.53, 37.6), turned to 0 degrees
- moved R9 36.6 mm to (14.1, 6.13), flipped to the bottom, turned to 270 degrees
- moved R2 35.1 mm to (25.2, 35.1)
- moved C6 31.7 mm to (29.6, 31.3)
- moved C7 31.5 mm to (26.3, 26.8), turned to 0 degrees
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- renumbered C27 to C19, LIPO to J1, SWITCH to SW1
Connections:
- removed net A4: U4.10
- removed net A5: U4.47
- removed net A5/SW2: IC1.3
- removed net BUZZ: Q2.1, R1.1
- removed net CS_3.3V: U3.13
- removed net D10: U4.27
- removed net D11/MOSI: U3.19
- removed net D13/SCK: U3.18
- removed net D2: U4.23
- removed net D5: U4.24
- removed net D6: U4.29
- removed net D7: U4.30
- removed net D8: U4.11
- removed net DC/SA0_3.3V: U3.15
- removed net LED: R8.1
- removed net N$8 (its old number): R15.1, S2.1
- removed net PHOTO: R10.2, R9.2
- removed net RST_3.3V: U3.14
- removed net SW1: C2.1, R4.2, S2.3
- removed net SW2: C1.1, R2.2, S1.3
- new net A4/PHOTO: R16.2, R17.2, U1.10
- new net A5/LED: R13.1, U1.47
- new net D10/OLED.CS: U1.27, U3.13
- new net D2/BUZZ: Q2.1, R11.1, U1.23
- new net D5/SW1: C20.1, OP1.3, R9.2, S1.3, U1.24
- new net D6/OLED.DC: U1.29, U3.15
- new net D7/SW2: C21.1, R10.2, S2.3, U1.30
- new net D8/OLED.RST: U1.11, U3.14
- new net N$12: R8.1, S2.1
- net !CS: now also U4.8; no longer ACCEL.8
- net !RESET: now also J2.10, R1.1, U1.40; no longer JP6.10, R11.1, U4.40
- net 3.3V: now also C10.1, C18.2, C22.1, C23.1, C4.1, J2.1, J3.2, LDO1.5, R1.2, R14.2, R16.1, R8.2, U1.17, U1.36, U1.44, U4.1, U4.14; no longer ACCEL.1, ACCEL.14, C12.1, C16.1, C18.1, C21.1, C29.2, JP6.1, LDO.5, LIS3DH.ACCEL.2, R10.1, R11.2, R5.2, R6.2, U4.17, U4.36, U4.44
- net 3V: now also C12.2, OP1.5; no longer C4.2, IC1.5
- net A0: now also U1.3; no longer U4.3
- net A1: now also U1.7; no longer U4.7
- net A2: now also U1.8; no longer U4.8
- net A3: now also U1.9; no longer U4.9
- net ADC1: now also U4.16; no longer ACCEL.16
- net ADC2: now also U4.15; no longer ACCEL.15
- net ADC3: now also U4.13; no longer ACCEL.13
- net AREF: now also U1.4; no longer U4.4
- net D0/RXI: now also U1.16; no longer U4.16
- net D1/TXO: now also U1.15; no longer U4.15
- net D11: now also U1.25; no longer U4.25
- net D12: now also U1.28; no longer U4.28
- net D13: now also U1.26; no longer U4.26
- net D3: now also U1.14; no longer U4.14
- net D4: now also U1.13; no longer U4.13
- net D9: now also U1.12; no longer U4.12
- net GND: now also C12.1, C13.1, C16.1, C18.1, C2.1, C20.2, C22.2, C23.2, C4.2, C5.2, C9.2, J2.3, J2.5, J3.1, LDO1.2, OP1.2, R10.1, R11.2, R17.1, R6.1, U1.18, U1.35, U1.42, U1.5, U2.2, U4.10, U4.12, U4.7, USB1.5, USB1.S1, USB1.S2, USB1.S3, USB1.S4, USB1.S5, USB1.S6; no longer ACCEL.10, ACCEL.12, ACCEL.5, ACCEL.7, C12.2, C15.2, C16.2, C17.2, C18.2, C2.2, C26.1, C28.1, C29.1, C4.1, C9.1, CHRG.2, IC1.2, JP6.3, JP6.5, LDO.2, LIS3DH.ACCEL.1, R1.2, R2.1, R22.1, R33.1, U$15.5, U$15.S1, U$15.S2, U$15.S3, U$15.S4, U$15.S5, U$15.S6, U4.18, U4.35, U4.42
- net INT1: now also U4.11; no longer ACCEL.11
- net INT2: now also U4.9; no longer ACCEL.9
- net N$14: now also U2.5; no longer CHRG.5
- net N$16: now also D1.-, D2.-; no longer D8.-, D9.-
- net N$17: now also C14.1, R5.1; no longer C3.1, R16.1
- net N$2: now also C2.2, U1.1; no longer C9.2, U4.1
- net N$22: now also R4.2; no longer R22.2
- net N$23: now also BUZZ1.-, D3.+; no longer D2.+, U$1.-
- net N$24: now also R6.2; no longer R33.2
- net N$25: now also C17.2; no longer C22.2
- net N$26: now also C17.1; no longer C22.1
- net N$27: now also C15.2; no longer C23.2
- net N$3: now also R13.2; no longer R8.2
- net N$38: now also C15.1; no longer C23.1
- net N$39: now also C13.2; no longer C26.2
- net N$4: now also C3.1, U1.2; no longer C7.1, U4.2
- net N$47: now also C16.2; no longer C28.2
- net N$7: now also OP1.1, OP1.4, R5.2; no longer IC1.1, IC1.4, R16.2
- net PA13: now also U1.22; no longer U4.22
- net PB22: now also U1.37; no longer U4.37
- net PB23: now also U1.38; no longer U4.38
- net RX_LED: now also U1.48; no longer U4.48
- net SCL: now also J3.4, R14.1, U1.32, U4.4; no longer ACCEL.4, LIS3DH.ACCEL.4, R5.1, U4.32
- net SDA: now also J3.3, R15.1, U1.31, U4.6; no longer ACCEL.6, LIS3DH.ACCEL.3, R6.1, U4.31
- net SPI_MISO: now also U1.21; no longer U4.21
- net SPI_MOSI: now also U1.19, U3.19; no longer U4.19
- net SPI_SCK: now also U1.20, U3.18; no longer U4.20
- net STAT: now also R2.1, U2.1; no longer CHRG.1, R13.1
- net SWCLK: now also J2.4, U1.45; no longer JP6.4, U4.45
- net SWDIO: now also J2.2, U1.46; no longer JP6.2, U4.46
- net TX_LED: now also U1.39; no longer U4.39
- net USB_D+: now also U1.34, USB1.3; no longer U$15.3, U4.34
- net USB_D-: now also U1.33, USB1.2; no longer U$15.2, U4.33
- net USB_HOST_EN: now also U1.41; no longer U4.41
- net V+: now also BUZZ1.+, D3.-; no longer D2.-, U$1.+
- net VDDANA: now also C1.1, U1.6; no longer C6.1, U4.6
- net VDDCORE: now also C5.1, U1.43; no longer C10.1, U4.43
- net VIN: now also C6.1, C7.1, LDO1.1, LDO1.3, R2.2, U2.4; no longer C14.1, C15.1, CHRG.4, LDO.1, LDO.3, R13.2
- net VLIPO: now also C9.1, D1.+, U2.3; no longer C17.1, CHRG.3, D8.+
- net V_USB: now also D2.+, USB1.1; no longer D9.+, U$15.1
Routing:
- net SDA: track 1.52 -> 43.0 mm, vias 0 -> 3
- net SCL: track 1.16 -> 39.9 mm, vias 0 -> 2
- net A4/PHOTO: track 0.00 -> 29.9 mm
- net VIN: track 0.00 -> 27.3 mm, vias 0 -> 3
- net USB_D-: track 0.00 -> 25.6 mm, vias 0 -> 2
- net !RESET: track 0.00 -> 25.0 mm, vias 0 -> 2
- net USB_D+: track 0.00 -> 24.5 mm, vias 0 -> 2
- net A5/LED: track 0.00 -> 21.1 mm, vias 0 -> 2
- net GND: track 0.00 -> 20.7 mm, vias 0 -> 13
- net D5/SW1: track 0.00 -> 20.6 mm
- net D7/SW2: track 0.00 -> 15.4 mm
- net 3.3V: track 12.1 -> 25.0 mm, vias 9 -> 16
- net D2/BUZZ: track 0.00 -> 12.8 mm
- net VLIPO: track 2.08 -> 13.6 mm
- net N$16: track 0.00 -> 10.8 mm, vias 0 -> 1
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Other:
- outline, holes or cut-outs redrawn
- board text added: "GERI Gadget"
