File: hardware/GERI_Gadget.sch (EAGLE design)
At the start: 62 parts, among them IC1 OP-SINGLEOT, Q1 5.8A/30V/35mΩ, Q2 5.8A/30V/35mΩ, U3 UG-2864HSWEG01, U4 ATSAMD21G-A, Y1 32.768kHz

Commit message: updates...almost done
Parts:
- removed ACCEL: LIS3DH, SparkFun-Sensors:LIS3DH
- removed C28, C29: 2.2uF, CalvEngIO-Passives:CAPACITOR0603
- removed D9: (no value), CalvEngIO-DiscreteSemi:SCHOTTKY-USC
- removed JP6: CORTEX_DEBUGPTH, samd21-temp:CORTEX_DEBUGPTH
- removed R22: 10K, CalvEngIO-Passives:RESISTOR0402-BIGGER
- removed R33: 390K, CalvEngIO-Passives:RESISTOR0402-BIGGER
- removed U$1: BUZZER_CMT-6635C-030, CalvEngIO-Electromechanical:BUZZER_CMT-6635C-030
- added BUZZ1: BUZZER.GENERIC, CalvEngIO-Electromechanical:BUZZER.GENERIC
- added C20: 100n, CalvEngIO-Passives:CAPACITOR0402
- added C5: 0.1uF, CalvEngIO-Passives:CAPACITOR0402
- added D3: (no value), CalvEngIO-DiscreteSemi:SCHOTTKY-USC
- added J2: CORTEX_DEBUG_PTH, CalvEngIO-Connectors:CORTEX_DEBUG_PTH
- added R14: 10k, SparkFun-Resistors:RESISTOR0402
- added R17: PHOTOCELLPTH, CalvEngIO-Sensors:PHOTOCELLPTH
- added REV1: REVISION.A, CalvEngIO-Logos:REVISION.A
- added U1: ATSAMD21G-A, CalvEngIO-Microcontrollers:ATSAMD21G-A
- C1: value 100n -> 0.1uF
- C12: value 0.1uF -> 100nF
- C14: value 10u -> 10uF
- C15, C16: value 2.2u -> 2.2uF
- C17: value 10u -> 2.2uF
- C18: value 0.1uF -> 2.2uF; device SparkFun-Capacitors:0.1UF-0402-16V-10% -> CalvEngIO-Passives:CAPACITOR0603
- C2: value 100n -> 15pF
- C21: value 10uF -> 100n; device SparkFun-Capacitors:10UF-0603-6.3V-20% -> CalvEngIO-Passives:CAPACITOR0402
- C22: value 2.2uF -> 0.1uF; device CalvEngIO-Passives:CAPACITOR0603 -> SparkFun-Capacitors:0.1UF-0402-16V-10%
- C23: value 2.2uF -> 10uF; device CalvEngIO-Passives:CAPACITOR0603 -> SparkFun-Capacitors:10UF-0603-6.3V-20%
- C3: value 10uF -> 15pF; device CalvEngIO-Passives:CAPACITOR0603 -> CalvEngIO-Passives:CAPACITOR0402
- C4: value 100nF -> 0.1uF
- C6: value 0.1uF -> 10u; device CalvEngIO-Passives:CAPACITOR0402 -> CalvEngIO-Passives:CAPACITOR0603
- C7: value 15pF -> 2.2u; device CalvEngIO-Passives:CAPACITOR0402 -> CalvEngIO-Passives:CAPACITOR0603
- C8: value 0.1uF -> 2.2u; device CalvEngIO-Passives:CAPACITOR0402 -> CalvEngIO-Passives:CAPACITOR0603
- C9: value 15pF -> 10u; device CalvEngIO-Passives:CAPACITOR0402 -> CalvEngIO-Passives:CAPACITOR0603
- R1: value 390k -> 10K
- R11: value 10K -> 390k
- R13: value 10k -> 1k
- R15: value 1k -> 10k; device CalvEngIO-Passives:RESISTOR0402-BIGGER -> SparkFun-Resistors:RESISTOR0402
- R16: value 390k -> 10k
- R4: value 10k -> 10K
- R5: value 10k -> 390k; device SparkFun-Resistors:RESISTOR0402 -> CalvEngIO-Passives:RESISTOR0402-BIGGER
- R6: value 10k -> 390K; device SparkFun-Resistors:RESISTOR0402 -> CalvEngIO-Passives:RESISTOR0402-BIGGER
- R9: value PHOTOCELLPTH -> 10k; device CalvEngIO-Sensors:PHOTOCELLPTH -> CalvEngIO-Passives:RESISTOR0402-BIGGER
- U4: value ATSAMD21G-A -> LIS3DH; device samd21-temp:ATSAMD21G-A -> SparkFun-Sensors:LIS3DH
- renumbered C26 to C13, C27 to C19, CHRG to U2, D8 to D1, IC1 to OP1, LDO to LDO1, LIPO to J1, LIS3DH.ACCEL to J3, SWITCH to SW1, U$15 to USB1
Connections:
- removed net A4: U4.PA05(AIN5/SER0:1/TC0:1)
- removed net A5: U4.PB02(AIN10/SER5:0)
- removed net A5/SW2: OP1G$1.+IN
- removed net BUZZ: Q2.G, R1.1
- removed net CS_3.3V: U3./CS
- removed net D10: U4.PA18(SER1:2+)
- removed net D11/MOSI: U3.D1/SPI_SDIN/I2C_SDA
- removed net D13/SCK: U3.D0/SPI_SCLK/I2C_SCK
- removed net D2: U4.PA14(XIN/SER2:2+)
- removed net D5: U4.PA15(XOUT/SER2:3+)
- removed net D6: U4.PA20(SER5:2+)
- removed net D7: U4.PA21(SER5:3+)
- removed net D8: U4.PA06(AIN6/SER0:2/TC1:0)
- removed net DC/SA0_3.3V: U3.DC/I2C_SA0
- removed net LED: R8.1
- removed net N$8 (its old number): R15.1, S2.1
- removed net PHOTO: R10.2, R9.P$2
- removed net RST_3.3V: U3./RES
- removed net SW1: C2.1, R4.2, S2.2
- removed net SW2: C1.1, R2.2, S1.2
- new net A4/PHOTO: R16.2, R17.P$2, U1.PA05(AIN5/SER0:1/TC0:1)
- new net A5/LED: R13.1, U1.PB02(AIN10/SER5:0)
- new net D10/OLED.CS: U1.PA18(SER1:2+), U3./CS
- new net D2/BUZZ: Q2.G, R11.1, U1.PA14(XIN/SER2:2+)
- new net D5/SW1: C20.1, OP1G$1.+IN, R9.2, S1.2, U1.PA15(XOUT/SER2:3+)
- new net D6/OLED.DC: U1.PA20(SER5:2+), U3.DC/I2C_SA0
- new net D7/SW2: C21.1, R10.2, S2.2, U1.PA21(SER5:3+)
- new net D8/OLED.RST: U1.PA06(AIN6/SER0:2/TC1:0), U3./RES
- new net N$12: R8.1, S2.1
- net !CS: now also U4.!CS!/MODE; no longer ACCEL.!CS!/MODE
- net !RESET: now also J2.!RESET, R1.1, U1.!RESET!; no longer JP6.NRESET, R11.1, U4.!RESET!
- net 3.3V: now also C10.1, C18.2, C22.1, C23.1, C4.1, J2.VCC, R1.2, R14.2, R16.1, R8.2, U1.VDDIN, U1.VDDIO@17, U1.VDDIO@36, U4.VDD, U4.VDDIO; no longer ACCEL.VDD, ACCEL.VDDIO, C12.1, C16.1, C18.1, C21.1, C29.2, JP6.VCC, R10.1, R11.2, R5.2, R6.2, U4.VDDIN, U4.VDDIO@17, U4.VDDIO@36
- net 3V: now also C12.2; no longer C4.2
- net A0: now also U1.PA02(AIN0/DAC); no longer U4.PA02(AIN0/DAC)
- net A1: now also U1.PB08(AIN2/SER4:0/TC4:0); no longer U4.PB08(AIN2/SER4:0/TC4:0)
- net A2: now also U1.PB09(AIN3/SER4:1/TC4:1); no longer U4.PB09(AIN3/SER4:1/TC4:1)
- net A3: now also U1.PA04(AIN4/REFB/SER0:0/TC0:0); no longer U4.PA04(AIN4/REFB/SER0:0/TC0:0)
- net ADC1: now also U4.ADC1; no longer ACCEL.ADC1
- net ADC2: now also U4.ADC2; no longer ACCEL.ADC2
- net ADC3: now also U4.ADC3; no longer ACCEL.ADC3
- net AREF: now also U1.PA03(AIN1/REFA); no longer U4.PA03(AIN1/REFA)
- net D0/RXI: now also U1.PA11(AIN19/SER0:3+); no longer U4.PA11(AIN19/SER0:3+)
- net D1/TXO: now also U1.PA10(AIN18/SER0:2+); no longer U4.PA10(AIN18/SER0:2+)
- net D11: now also U1.PA16(I2C/SER1:0+); no longer U4.PA16(I2C/SER1:0+)
- net D12: now also U1.PA19(SER1:3+); no longer U4.PA19(SER1:3+)
- net D13: now also U1.PA17(I2C/SER1:1+); no longer U4.PA17(I2C/SER1:1+)
- net D3: now also U1.PA09(I2C/AIN17/SER0:1+); no longer U4.PA09(I2C/AIN17/SER0:1+)
- net D4: now also U1.PA08(I2C/AIN16/SER0:0+); no longer U4.PA08(I2C/AIN16/SER0:0+)
- net D9: now also U1.PA07(AIN7/SER0:3/TC1:1); no longer U4.PA07(AIN7/SER0:3/TC1:1)
- net GND: now also C12.1, C16.1, C18.1, C2.1, C20.2, C22.2, C23.2, C4.2, C5.2, C9.2, J2.GND@3, J2.GND@5, R10.1, R11.2, R17.P$1, R6.1, R9.1, U1.GND@18, U1.GND@35, U1.GND@42, U1.GNDANA, U4.GND@12, U4.GND@5, U4.RES, U4.SA0/SDO; no longer ACCEL.GND@12, ACCEL.GND@5, ACCEL.RES, ACCEL.SA0/SDO, C12.2, C15.2, C16.2, C17.2, C18.2, C2.2, C28.1, C29.1, C4.1, C9.1, JP6.GND@3, JP6.GND@5, R1.2, R2.1, R22.1, R33.1, R9.P$1, U4.GND@18, U4.GND@35, U4.GND@42, U4.GNDANA
- net INT1: now also U4.INT1; no longer ACCEL.INT1
- net INT2: now also U4.INT2; no longer ACCEL.INT2
- net N$16: now also D2.C; no longer D9.C
- net N$17: now also C14.1, R5.1; no longer C3.1, R16.1
- net N$2: now also C2.2, U1.PA00(XIN32/SER1:0/TC2:0); no longer C9.2, U4.PA00(XIN32/SER1:0/TC2:0)
- net N$22: now also R4.2; no longer R22.2
- net N$23: now also BUZZ1.-, D3.A; no longer D2.A, U$1.-
- net N$24: now also R6.2; no longer R33.2
- net N$25: now also C17.2; no longer C22.2
- net N$26: now also C17.1; no longer C22.1
- net N$27: now also C15.2; no longer C23.2
- net N$3: now also R13.2; no longer R8.2
- net N$38: now also C15.1; no longer C23.1
- net N$4: now also C3.1, U1.PA01(XOUT32/SER1:1/TC2:1); no longer C7.1, U4.PA01(XOUT32/SER1:1/TC2:1)
- net N$47: now also C16.2; no longer C28.2
- net N$7: now also R5.2; no longer R16.2
- net PA13: now also U1.PA13(I2C/SER2:1+); no longer U4.PA13(I2C/SER2:1+)
- net PB22: now also U1.PB22(SER5:2+); no longer U4.PB22(SER5:2+)
- net PB23: now also U1.PB23(SER5:3+); no longer U4.PB23(SER5:3+)
- net RX_LED: now also U1.PB03(AIN11/SER5:1); no longer U4.PB03(AIN11/SER5:1)
- net SCL: now also R14.1, U1.PA23(I2C/SER3:0+), U4.SCL/SPC; no longer ACCEL.SCL/SPC, R5.1, U4.PA23(I2C/SER3:0+)
- net SDA: now also R15.1, U1.PA22(I2C/SER3:0+), U4.SDA/SDI; no longer ACCEL.SDA/SDI, R6.1, U4.PA22(I2C/SER3:0+)
- net SPI_MISO: now also U1.PA12(I2C/SER2:0+); no longer U4.PA12(I2C/SER2:0+)
- net SPI_MOSI: now also U1.PB10(SER4:2+), U3.D1/SPI_SDIN/I2C_SDA; no longer U4.PB10(SER4:2+)
- net SPI_SCK: now also U1.PB11(SER4:3+), U3.D0/SPI_SCLK/I2C_SCK; no longer U4.PB11(SER4:3+)
- net STAT: now also R2.1; no longer R13.1
- net SWCLK: now also J2.SWDCLK/TCK, U1.PA30(SWCLK/SER1:2+); no longer JP6.SWDCLK/TCK, U4.PA30(SWCLK/SER1:2+)
- net SWDIO: now also J2.SWDIO/TMS, U1.PA31(SWDIO/SER1:3+); no longer JP6.SWDIO/TMS, U4.PA31(SWDIO/SER1:3+)
- net TX_LED: now also U1.PA27; no longer U4.PA27
- net USB_D+: now also U1.PA25(SER3:3+); no longer U4.PA25(SER3:3+)
- net USB_D-: now also U1.PA24(SER3:2+); no longer U4.PA24(SER3:2+)
- net USB_HOST_EN: now also U1.PA28; no longer U4.PA28
- net V+: now also BUZZ1.+, D3.C; no longer D2.C, U$1.+
- net VDDANA: now also C1.1, U1.VDDANA; no longer C6.1, U4.VDDANA
- net VDDCORE: now also C5.1, U1.VDDCORE; no longer C10.1, U4.VDDCORE
- net VIN: now also C6.1, C7.1, R2.2; no longer C14.1, C15.1, R13.2
- net VLIPO: now also C9.1; no longer C17.1
- net V_USB: now also D2.A; no longer D9.A
Other:
- note added: "GERI Gadget"
- note removed: "Have to switch the default SPI pins"
- moved on the sheet: C1, C10, C11, C12, C14, C15, C16, C17, C18, C2, C21, C22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
